File: samo4k-pcb-test.kicad_pcb (KiCad board)
At the start: 2 copper layers, 80.2 x 38.1 mm, 24 parts, among them SW1 SW_Push, U1 ATmega32U4-AU, Y1 16MHz

Commit message: silks
Parts:
- moved C2 0.79 mm to (139.7, 61.9)
- moved R3 0.79 mm to (136.5, 61.9)
- moved USB1 0.54 mm to (127.0, 52.6)
Routing:
- net Net-(USB1-Pad6): track 0.00 -> 16.3 mm
- net Net-(R3-Pad2): track 45.8 -> 43.3 mm
- net COL1: track 35.7 -> 38.1 mm
- net COL0: track 41.6 -> 43.9 mm
- net D+: track 4.73 -> 6.66 mm
- net GND: track 129.8 -> 131.7 mm, vias 2 -> 4
- net VCC: track 18.4 -> 17.5 mm, vias 0 -> 2
- net +5V: track 128.3 -> 129.1 mm
- added copper zone on B.Cu, net GND
Other:
- outline, holes or cut-outs redrawn
- board text added: "made by kumots"
- board text added: "pagsamo 4k"
